Commit message: Yoink + Get working movie robot (throws itself)

File: body.urdf (robot description, URDF)
Before this commit: robot robot, 2 links, 1 joints
Links:
- removed link Foot
- added link leftCrutch, mass 1; collision box size=1 1 0.5; visual box size=1 1 0.5
- added link leftFoot, mass 1; collision box size=1 1 0.5; visual box size=1 1 0.5
- added link rightCrutch, mass 1; collision box size=1 1 0.5; visual box size=1 1 0.5
- added link rightFoot, mass 1; collision box size=1 1 1; visual box size=1 1 1
Joints:
- removed joint Foot_Torso
- added joint leftCrutch_Torso: type revolute, parent Torso, child leftCrutch, origin xyz=0 0.5 1 rpy=0 0 0, axis 0 1 0, limit lower=-3.14159 upper=3.14159 effort=0.0 velocity=0.0
- added joint leftFoot_Torso: type continuous, parent Torso, child leftFoot, origin xyz=0.5 0 1 rpy=0 0 0, axis 0 1 0, limit lower=-3.14159 upper=3.14159 effort=0.0 velocity=0.0
- added joint rightCrutch_Torso: type revolute, parent Torso, child rightCrutch, origin xyz=0 -0.5 1 rpy=0 0 0, axis 0 1 0, limit lower=-3.14159 upper=3.14159 effort=0.0 velocity=0.0
- added joint rightFoot_Torso: type revolute, parent Torso, child rightFoot, origin xyz=-0.5 0 1 rpy=0 0 0, axis 0 1 0, limit lower=-3.14159 upper=3.14159 effort=0.0 velocity=0.0
